Commit message: changed collision box of raybot to correct size

File: Plankton/raybot_description/urdf/raybot_base.xacro (robot description, xacro)
@@ -33,4 +33,5 @@
   <xacro:property name="namespace" value="raybot"/>
   <xacro:property name="visual_mesh_file" value="file://$(find raybot_description)/meshes/frame_kolom_origin_com.dae"/>
+  <xacro:property name="collision_mesh_file" value="file://$(find raybot_description)/meshes/frame_collision_origin_com.dae"/>
   <xacro:property name="prop_mesh_file" value="file://$(find raybot_description)/meshes/prop.dae"/>
   <!-- Mass, see p.28 in Berg2012 -->
@@ -52,22 +53,8 @@
       <!-- bottom plate -->
       <collision>
-        <origin xyz="0 0 -0.75" rpy="0 0 0"/>
+        <origin xyz="0 0 0" rpy="1.5708 0 3.1416"/>
         <geometry>
-          <box size="2.56 1.50 0.10"/>
+          <mesh filename="${collision_mesh_file}" scale="1 1 1"/>
         </geometry>
-      </collision>
-      <!-- top plate -->
-      <collision>
-        <origin xyz="0 0 0.60" rpy="0 0 0"/>
-        <geometry><box size="2.56 1.50 0.40"/></geometry>
-      </collision>
-      <!-- left / right sides -->
-      <collision>
-        <origin xyz="-0.20 0.70 -0.15" rpy="0 0 0"/>
-        <geometry><box size="2.20 0.10 1.10"/></geometry>
-      </collision>
-      <collision>
-        <origin xyz="-0.20 -0.70 -0.15" rpy="0 0 0"/>
-        <geometry><box size="2.20 0.10 1.10"/></geometry>
       </collision>
     </link>
