Commit message: commit with pid and mpc

File: Plankton/raybot_description/urdf/raybot.gazebo.xacro (robot description, xacro)
@@ -25,5 +25,5 @@
     <xacro:property name="cob" value="0.0 0.0 0.2"/> <!--- "0.0 0.0 0.3" -->
     <!-- Volume, see p.31 in Berg2012 -->
-    <xacro:property name="volume" value="0.04089"/> <!-- 1.83826  of 0.168 xxxxxxxxxxxxxxxxxxxxxxxxxxxxxxxxxxxxxxxxxxxxxxxxxxxxxxxxxxxxxxxxxxxxxxxxxxxxxxxxxxxxxxxxxxxxxxxxxxxxxxxxxxxx -->
+    <xacro:property name="volume" value="0.02633"/> <!-- 1.83826  of 0.168 xxxxxxxxxxxxxxxxxxxxxxxxxxxxxxxxxxxxxxxxxxxxxxxxxxxxxxxxxxxxxxxxxxxxxxxxxxxxxxxxxxxxxxxxxxxxxxxxxxxxxxxxxxxx -->
     <xacro:macro name="raybot_hydro_model" params="namespace">
         <link name="${namespace}/base_link">
@@ -31,7 +31,7 @@
             <volume>${volume}</volume>
             <box>
-                <width>0.8</width> <!-- 1.5 xxxxxxxxxxxxxxxxxxxxxxxxxxxxxxxxxxxxxxxxxxxxxxxxxxxxxxxxxxxxxxxxxxxxxxxxxxxxxxxxxxxxxxxxxxxxxxxxxxxxxxxxxxxx -->
-                <length>0.28</length> <!-- 2.6 xxxxxxxxxxxxxxxxxxxxxxxxxxxxxxxxxxxxxxxxxxxxxxxxxxxxxxxxxxxxxxxxxxxxxxxxxxxxxxxxxxxxxxxxxxxxxxxxxxxxxxxxxxxx -->
-                <height>0.56</height> <!-- 1.6 xxxxxxxxxxxxxxxxxxxxxxxxxxxxxxxxxxxxxxxxxxxxxxxxxxxxxxxxxxxxxxxxxxxxxxxxxxxxxxxxxxxxxxxxxxxxxxxxxxxxxxxxxxxx -->
+                <width>1.21</width> <!-- 1.5 of 0.8 xxxxxxxxxxxxxxxxxxxxxxxxxxxxxxxxxxxxxxxxxxxxxxxxxxxxxxxxxxxxxxxxxxxxxxxxxxxxxxxxxxxxxxxxxxxxxxxxxxxxxxxxxxxx -->
+                <length>0.33</length> <!-- 2.6 of 0.28 xxxxxxxxxxxxxxxxxxxxxxxxxxxxxxxxxxxxxxxxxxxxxxxxxxxxxxxxxxxxxxxxxxxxxxxxxxxxxxxxxxxxxxxxxxxxxxxxxxxxxxxxxxxx -->
+                <height>0.59</height> <!-- 1.6 of 0.56 xxxxxxxxxxxxxxxxxxxxxxxxxxxxxxxxxxxxxxxxxxxxxxxxxxxxxxxxxxxxxxxxxxxxxxxxxxxxxxxxxxxxxxxxxxxxxxxxxxxxxxxxxxxx -->
             </box>
             <center_of_buoyancy>${cob}</center_of_buoyancy>
@@ -51,5 +51,5 @@
                     0 0 0 1 0 1
                     0 0 0 0 1 0
-                    0 0 0 0 0 1  -->
+                    0 0 0 0 0 1
                     53.56 0    0    0     0     0
                     0     10.3 0    0     0     0
@@ -57,15 +57,21 @@
                     0     0    0    0.784 0     0
                     0     0    0    0     0.564 0
-                    0     0    0    0     0     1.367
+                    0     0    0    0     0     1.367 -->
+                    27.96 0     0     0     0     0
+                    0     20.35 0     0     0     0
+                    0     0     29.58 0     0     0
+                    0     0     0     3.90  0     0
+                    0     0     0     0     1.48  0
+                    0     0     0     0     0     4.06
                 </added_mass>
                 <!-- Linear damping: see p.31 in Berg2012 -->
                 <linear_damping>
                   <!--  -74.82 -69.48 -728.4 -268.8 -309.77 -105 -->
-                  -4 -6 -5 -0.07 -0.07 -0.07
+                  -24.65 -56.70 -47.01 -0.0312 -0.07 -2.956
                 </linear_damping>
                 <!-- Non-linear damping: see p.30 in Berg2012 -->
                 <quadratic_damping>
                    <!-- -748.22 -992.53 -1821.01 -672 -774.44 -523.27 -->
-                   -18 -21 -37 -1.5 -1.5 -1.5
+                   -747.06 -181.73 -681.28 -1.9088 -1 -0.133
                 </quadratic_damping>
             </hydrodynamic_model>

File: Plankton/raybot_description/urdf/raybot_actuators.xacro (robot description, xacro)
@@ -18,5 +18,5 @@
 -->
 <robot xmlns:xacro="http://www.ros.org/wiki/xacro">
-  <xacro:property name="prop_mesh_file" value="file://$(find raybot_description)/meshes/raybot_simple_thruster_v2.dae"/>
+  <xacro:property name="prop_mesh_file" value="file://$(find raybot_description)/meshes/T200_thruster_simple.dae"/>
   <!-- Thruster joint and link snippet -->
   <xacro:macro name="thruster_macro"
@@ -32,26 +32,26 @@
   </xacro:macro>
   <xacro:thruster_macro namespace="${namespace}" thruster_id="0">
-   <origin xyz="0 -0.34 0.21" rpy="${0*d2r} ${0*d2r} ${0*d2r}"/>
+   <origin xyz="0 -0.51 0.20" rpy="${0*d2r} ${0*d2r} ${0*d2r}"/>
   </xacro:thruster_macro>
   <xacro:thruster_macro namespace="${namespace}" thruster_id="1">
-   <origin xyz="0 0.34 0.21" rpy="${0*d2r} ${0*d2r} ${0*d2r}"/>
+   <origin xyz="0 0.51 0.20" rpy="${0*d2r} ${0*d2r} ${0*d2r}"/>
   </xacro:thruster_macro>
   <xacro:thruster_macro namespace="${namespace}" thruster_id="2">
-   <origin xyz="0 0.34 -0.21" rpy="${0*d2r} ${0*d2r} ${0*d2r}"/>
+   <origin xyz="0 0.51 -0.20" rpy="${0*d2r} ${0*d2r} ${0*d2r}"/>
   </xacro:thruster_macro>
   <xacro:thruster_macro namespace="${namespace}" thruster_id="3">
-   <origin xyz="0 -0.34 -0.21" rpy="${0*d2r} ${0*d2r} ${0*d2r}"/>
+   <origin xyz="0 -0.51 -0.20" rpy="${0*d2r} ${0*d2r} ${0*d2r}"/>
   </xacro:thruster_macro>
   <xacro:thruster_macro namespace="${namespace}" thruster_id="4">
-   <origin xyz="0 0 0.21" rpy="${0*d2r} ${0*d2r} ${90.0*d2r}"/>
+   <origin xyz="0 0 0.20" rpy="${0*d2r} ${0*d2r} ${90.0*d2r}"/>
   </xacro:thruster_macro>
   <xacro:thruster_macro namespace="${namespace}" thruster_id="5">
-   <origin xyz="0 0 -0.21" rpy="${0*d2r} ${0*d2r} ${90.0*d2r}"/>
+   <origin xyz="0 0 -0.20" rpy="${0*d2r} ${0*d2r} ${90.0*d2r}"/>
   </xacro:thruster_macro>
   <xacro:thruster_macro namespace="${namespace}" thruster_id="6">
-   <origin xyz="0 0.34 0" rpy="${0*d2r} ${-90*d2r} ${0*d2r}"/>
+   <origin xyz="0 0.51 0" rpy="${0*d2r} ${-90*d2r} ${0*d2r}"/>
   </xacro:thruster_macro>
   <xacro:thruster_macro namespace="${namespace}" thruster_id="7">
-   <origin xyz="0 -0.34 0" rpy="${0*d2r} ${-90*d2r} ${0*d2r}"/>
+   <origin xyz="0 -0.51 0" rpy="${0*d2r} ${-90*d2r} ${0*d2r}"/>
   </xacro:thruster_macro>
 </robot>

File: Plankton/raybot_description/urdf/raybot_base.xacro (robot description, xacro)
@@ -32,9 +32,9 @@
   <!-- Parameters -->
   <xacro:property name="namespace" value="raybot"/>
-  <xacro:property name="visual_mesh_file" value="file://$(find raybot_description)/meshes/raybot_simple_frame_water_v2.dae"/>
-  <xacro:property name="collision_mesh_file" value="file://$(find raybot_description)/meshes/raybot_simple_collision_v2.dae"/>
-  <xacro:property name="prop_mesh_file" value="file://$(find raybot_description)/meshes/raybot_simple_thruster_v2.dae"/>
+  <xacro:property name="visual_mesh_file" value="file://$(find raybot_description)/meshes/assembly_raybot_simple_without_thrusters.dae"/>
+  <xacro:property name="collision_mesh_file" value="file://$(find raybot_description)/meshes/raybot_collision.dae"/>
+  <xacro:property name="prop_mesh_file" value="file://$(find raybot_description)/meshes/T200-THRUSTER-R1_propellor.dae"/>
   <!-- Mass, see p.28 in Berg2012 -->
-  <xacro:property name="mass" value="40.89"/> <!-- 1862.87 of 168 xxxxxxxxxxxxxxxxxxxxxxxxxxxxxxxxxxxxxxxxxxxxxxxxxxxxxxxxxxxxxxxxxxxxxxxxxxxxxxxxxxxxxxxxxxxxxx -->
+  <xacro:property name="mass" value="26.33"/> <!-- 1862.87 of 168 xxxxxxxxxxxxxxxxxxxxxxxxxxxxxxxxxxxxxxxxxxxxxxxxxxxxxxxxxxxxxxxxxxxxxxxxxxxxxxxxxxxxxxxxxxxxxx -->
   <xacro:macro name="raybot_base" params="namespace *gazebo inertial_reference_frame">
     <!-- base_link according to ROS conventions: x forward, z up -->
@@ -43,5 +43,5 @@
         <mass value="${mass}"/>
         <origin xyz="0 0 0"/>
-        <inertia ixx="3.04999" ixy="0" ixz="0" iyy="1.19804" iyz="0" izz="2.36173"/> <!--ixx="1.19804" ixy="0" ixz="0.00124" iyy="2.36173" iyz="0" izz="3.04999" of  ixx="525.39" ixy="1.44" ixz="33.41" iyy="794.20" iyz="2.6" izz="691.23"/> of ixx="23.66" ixy="0" ixz="0" iyy="21.25" iyz="0" izz="4.6" xxxxxxxxxxxxxxxxx -->
+        <inertia ixx="6.28" ixy="0" ixz="0" iyy="1.96" iyz="0" izz="5.32"/> <!--ixx="1.19804" ixy="0" ixz="0.00124" iyy="2.36173" iyz="0" izz="3.04999" of  ixx="525.39" ixy="1.44" ixz="33.41" iyy="794.20" iyz="2.6" izz="691.23"/> of ixx="23.66" ixy="0" ixz="0" iyy="21.25" iyz="0" izz="4.6" xxxxxxxxxxxxxxxxx -->
       </inertial>
       <visual>

File: Plankton/raybot_description/urdf/raybot_sensors.xacro (robot description, xacro)
@@ -36,5 +36,5 @@
   </xacro:default_pressure_macro> -->
   <!-- IMU  -->
-  <xacro:default_imu_macro
+ <xacro:default_imu_macro
     namespace="${namespace}"
     parent_link="${namespace}/base_link"

File: Plankton/uuv_sensor_plugins/uuv_sensor_ros_plugins/urdf/magnetometer_snippets.xacro (robot description, xacro)
@@ -59,5 +59,5 @@
       <visual>
         <geometry>
-          <box size="0.1 0.1 0.1" />
+          <box size="0.0001 0.0001 0.0001" />
         </geometry>
       </visual>

Commit message: updated commit with ERK4

File: Plankton/raybot_description/urdf/raybot.gazebo.xacro (robot description, xacro)
@@ -23,10 +23,10 @@
     assume NWU (otherwise cob is below cog?).
     -->
-    <xacro:property name="cob" value="0.0 0.0 0.2"/> <!--- "0.0 0.0 0.3" -->
+    <xacro:property name="cob" value="0.0 0.0 0.3"/> <!--- "0.0 0.0 0.3" of eerst ook nog "0.0 0.0 0.2" -->
     <!-- Volume, see p.31 in Berg2012 -->
-    <xacro:property name="volume" value="0.02633"/> <!-- 1.83826  of 0.168 xxxxxxxxxxxxxxxxxxxxxxxxxxxxxxxxxxxxxxxxxxxxxxxxxxxxxxxxxxxxxxxxxxxxxxxxxxxxxxxxxxxxxxxxxxxxxxxxxxxxxxxxxxxx -->
+    <xacro:property name="volume" value="0.02573"/> <!-- 1.83826  of 0.168 xxxxxxxxxxxxxxxxxxxxxxxxxxxxxxxxxxxxxxxxxxxxxxxxxxxxxxxxxxxxxxxxxxxxxxxxxxxxxxxxxxxxxxxxxxxxxxxxxxxxxxxxxxxx -->
     <xacro:macro name="raybot_hydro_model" params="namespace">
         <link name="${namespace}/base_link">
-            <neutrally_buoyant>1</neutrally_buoyant> <!-- 0 xxxxxxxxxxxxxxxxxxxxxxxxxxxxxxxxxxxxxxxxxxxxxxxxxxxxxxxxxxxxxxxxxxxxxxxxxxxxxxxxxxxxxxxxxxxxxxxxxxxxx -->
+            <neutrally_buoyant>0</neutrally_buoyant> <!-- 0 xxxxxxxxxxxxxxxxxxxxxxxxxxxxxxxxxxxxxxxxxxxxxxxxxxxxxxxxxxxxxxxxxxxxxxxxxxxxxxxxxxxxxxxxxxxxxxxxxxxxx -->
             <volume>${volume}</volume>
             <box>
@@ -58,20 +58,20 @@
                     0     0    0    0     0.564 0
                     0     0    0    0     0     1.367 -->
-                    27.96 0     0     0     0     0
-                    0     20.35 0     0     0     0
-                    0     0     29.58 0     0     0
-                    0     0     0     3.90  0     0
-                    0     0     0     0     1.48  0
-                    0     0     0     0     0     4.06
+                    27.96 0.0 0.0 0.0 0.0 0.0
+                    0.0 20.35 0.0 0.0 0.0 0.0
+                    0.0 0.0 29.58 0.0 0.0 0.0
+                    0.0 0.0 0.0 3.90  0.0 0.0
+                    0.0 0.0 0.0 0.0 1.48  0.0
+                    0.0 0.0 0.0 0.0 0.0 4.06
                 </added_mass>
                 <!-- Linear damping: see p.31 in Berg2012 -->
                 <linear_damping>
                   <!--  -74.82 -69.48 -728.4 -268.8 -309.77 -105 -->
-                  -24.65 -56.70 -47.01 -0.0312 -0.07 -2.956
+                  -24.65 -56.70 -47.01 -0.0312 -0.07 -0.2956
                 </linear_damping>
                 <!-- Non-linear damping: see p.30 in Berg2012 -->
                 <quadratic_damping>
                    <!-- -748.22 -992.53 -1821.01 -672 -774.44 -523.27 -->
-                   -747.06 -181.73 -681.28 -1.9088 -1 -0.133
+                   -747.06 -181.73 -681.28 -1.9088 -1 -1.33
                 </quadratic_damping>
             </hydrodynamic_model>

File: Plankton/raybot_description/urdf/raybot_base.xacro (robot description, xacro)
@@ -43,5 +43,5 @@
         <mass value="${mass}"/>
         <origin xyz="0 0 0"/>
-        <inertia ixx="6.28" ixy="0" ixz="0" iyy="1.96" iyz="0" izz="5.32"/> <!--ixx="1.19804" ixy="0" ixz="0.00124" iyy="2.36173" iyz="0" izz="3.04999" of  ixx="525.39" ixy="1.44" ixz="33.41" iyy="794.20" iyz="2.6" izz="691.23"/> of ixx="23.66" ixy="0" ixz="0" iyy="21.25" iyz="0" izz="4.6" xxxxxxxxxxxxxxxxx -->
+        <inertia ixx="6.28" ixy="0.0" ixz="0.0" iyy="1.96" iyz="0.0" izz="5.32"/> <!--ixx="1.19804" ixy="0" ixz="0.00124" iyy="2.36173" iyz="0" izz="3.04999" of  ixx="525.39" ixy="1.44" ixz="33.41" iyy="794.20" iyz="2.6" izz="691.23"/> of ixx="23.66" ixy="0" ixz="0" iyy="21.25" iyz="0" izz="4.6" xxxxxxxxxxxxxxxxx -->
       </inertial>
       <visual>

File: Plankton/uuv_descriptions/urdf/rexrov.gazebo.xacro (robot description, xacro)
@@ -25,5 +25,5 @@
     <xacro:property name="cob" value="0.0 0.0 0.3"/>
     <!-- Volume, see p.31 in Berg2012 -->
-    <xacro:property name="volume" value="1.83826"/>
+    <xacro:property name="volume" value="1.81"/> <!-- 1.83826 -->
     <xacro:macro name="rexrov_hydro_model" params="namespace">
         <link name="${namespace}/base_link">

File: Plankton/uuv_descriptions/urdf/rexrov_base.xacro (robot description, xacro)
@@ -35,5 +35,5 @@
   <xacro:property name="prop_mesh_file" value="file://$(find uuv_descriptions)/meshes/prop.dae"/>
   <!-- Mass, see p.28 in Berg2012 -->
-  <xacro:property name="mass" value="1862.87"/>
+  <xacro:property name="mass" value="1862.87"/> <!-- 1862.87 -->
   <xacro:macro name="rexrov_base" params="namespace *gazebo inertial_reference_frame">
     <!-- base_link according to ROS conventions: x forward, z up -->

File: Plankton/uuv_sensor_plugins/uuv_sensor_ros_plugins/urdf/pose_3d_snippets.xacro (robot description, xacro)
@@ -24,5 +24,5 @@
       <inertial>
         <inertia ixx="0.00001" ixy="0.0" ixz="0.0" iyy="0.00001" iyz="0.0" izz="0.00001" />
-        <mass value="0.001" />  <!-- [kg] -->
+        <mass value="0.01" />  <!-- [kg] -->
         <origin xyz="0 0 0" rpy="0 0 0" />
       </inertial>
