Commit message: changed raybot layout to vertical movement layout, /w added mass and correct inertia

File: Plankton/raybot_description/robots/raybot_default.xacro (robot description, xacro)
@@ -32,5 +32,5 @@
     <gazebo>
       <plugin name="$(arg namespace)_uuv_plugin" filename="libuuv_underwater_object_ros_plugin.so">
-        <fluid_density>1028.0</fluid_density>
+        <fluid_density>1025.0</fluid_density>
         <flow_velocity_topic>hydrodynamics/current_velocity</flow_velocity_topic>
         <debug>$(arg debug)</debug>

File: Plankton/raybot_description/urdf/raybot.gazebo.xacro (robot description, xacro)
@@ -23,15 +23,15 @@
     assume NWU (otherwise cob is below cog?).
     -->
-    <xacro:property name="cob" value="0.0 0.0 0.3"/>
+    <xacro:property name="cob" value="0.0 0.0 0.2"/> <!--- "0.0 0.0 0.3" -->
     <!-- Volume, see p.31 in Berg2012 -->
-    <xacro:property name="volume" value="1.83826"/>
+    <xacro:property name="volume" value="0.04089"/> <!-- 1.83826  of 0.168 xxxxxxxxxxxxxxxxxxxxxxxxxxxxxxxxxxxxxxxxxxxxxxxxxxxxxxxxxxxxxxxxxxxxxxxxxxxxxxxxxxxxxxxxxxxxxxxxxxxxxxxxxxxx -->
     <xacro:macro name="raybot_hydro_model" params="namespace">
         <link name="${namespace}/base_link">
-            <neutrally_buoyant>0</neutrally_buoyant>
+            <neutrally_buoyant>1</neutrally_buoyant> <!-- 0 xxxxxxxxxxxxxxxxxxxxxxxxxxxxxxxxxxxxxxxxxxxxxxxxxxxxxxxxxxxxxxxxxxxxxxxxxxxxxxxxxxxxxxxxxxxxxxxxxxxxx -->
             <volume>${volume}</volume>
             <box>
-                <width>1.5</width>
-                <length>2.6</length>
-                <height>1.6</height>
+                <width>0.8</width> <!-- 1.5 xxxxxxxxxxxxxxxxxxxxxxxxxxxxxxxxxxxxxxxxxxxxxxxxxxxxxxxxxxxxxxxxxxxxxxxxxxxxxxxxxxxxxxxxxxxxxxxxxxxxxxxxxxxx -->
+                <length>0.28</length> <!-- 2.6 xxxxxxxxxxxxxxxxxxxxxxxxxxxxxxxxxxxxxxxxxxxxxxxxxxxxxxxxxxxxxxxxxxxxxxxxxxxxxxxxxxxxxxxxxxxxxxxxxxxxxxxxxxxx -->
+                <height>0.56</height> <!-- 1.6 xxxxxxxxxxxxxxxxxxxxxxxxxxxxxxxxxxxxxxxxxxxxxxxxxxxxxxxxxxxxxxxxxxxxxxxxxxxxxxxxxxxxxxxxxxxxxxxxxxxxxxxxxxxx -->
             </box>
             <center_of_buoyancy>${cob}</center_of_buoyancy>
@@ -40,5 +40,5 @@
                 <!-- Added mass: see p.28 in Berg2012 -->
                 <added_mass>
-                     779.79 -6.8773 -103.32  8.5426 -165.54 -7.8033
+                 <!--    779.79 -6.8773 -103.32  8.5426 -165.54 -7.8033
                     -6.8773    1222   51.29  409.44 -5.8488  62.726
                     -103.32   51.29  3659.9  6.1112 -386.42  10.774
@@ -46,12 +46,26 @@
                     -165.54 -5.8488 -386.42 -10.027  842.69 -1.1162
                     -7.8033  62.726  10.775  21.019 -1.1162  224.32
+                    50 0 0 0 0 0
+                    0 40 0 0 0 0
+                    0 0 30 0 0 0
+                    0 0 0 1 0 1
+                    0 0 0 0 1 0
+                    0 0 0 0 0 1  -->
+                    53.56 0    0    0     0     0
+                    0     10.3 0    0     0     0
+                    0     0    23.6 0     0     0
+                    0     0    0    0.784 0     0
+                    0     0    0    0     0.564 0
+                    0     0    0    0     0     1.367
                 </added_mass>
                 <!-- Linear damping: see p.31 in Berg2012 -->
                 <linear_damping>
-                    -74.82 -69.48 -728.4 -268.8 -309.77 -105
+                  <!--  -74.82 -69.48 -728.4 -268.8 -309.77 -105 -->
+                  -4 -6 -5 -0.07 -0.07 -0.07
                 </linear_damping>
                 <!-- Non-linear damping: see p.30 in Berg2012 -->
                 <quadratic_damping>
-                    -748.22 -992.53 -1821.01 -672 -774.44 -523.27
+                   <!-- -748.22 -992.53 -1821.01 -672 -774.44 -523.27 -->
+                   -18 -21 -37 -1.5 -1.5 -1.5
                 </quadratic_damping>
             </hydrodynamic_model>

File: Plankton/raybot_description/urdf/raybot_actuators.xacro (robot description, xacro)
@@ -18,5 +18,5 @@
 -->
 <robot xmlns:xacro="http://www.ros.org/wiki/xacro">
-  <xacro:property name="prop_mesh_file" value="file://$(find raybot_description)/meshes/t200_thruster_blueesc_origin_tip.dae"/>
+  <xacro:property name="prop_mesh_file" value="file://$(find raybot_description)/meshes/raybot_simple_thruster_v2.dae"/>
   <!-- Thruster joint and link snippet -->
   <xacro:macro name="thruster_macro"
@@ -27,31 +27,31 @@
       mesh_filename="${prop_mesh_file}"
       dyn_time_constant="0.05"
-      rotor_constant="0.00031">
+      rotor_constant="0.0000033"> <!-- 0.00031 xxxxxxxxxxxxxxxxxxxxxxxxxxxxxxxxxxxxxxxxxxxxxxxxxxxxxxxxxxxxxxxxxxxxxxxxxxxxxxxxxxxxxxxxxxx -->
       <xacro:insert_block name="origin"/>
     </xacro:thruster_module_first_order_basic_fcn_macro>
   </xacro:macro>
   <xacro:thruster_macro namespace="${namespace}" thruster_id="0">
-   <origin xyz="0.14 -0.18515 0.549" rpy="${0*d2r} ${0*d2r} ${0*d2r}"/>
+   <origin xyz="0 -0.34 0.21" rpy="${0*d2r} ${0*d2r} ${0*d2r}"/>
   </xacro:thruster_macro>
   <xacro:thruster_macro namespace="${namespace}" thruster_id="1">
-   <origin xyz="0.14 0.18515 0.549" rpy="${0*d2r} ${0*d2r} ${0*d2r}"/>
+   <origin xyz="0 0.34 0.21" rpy="${0*d2r} ${0*d2r} ${0*d2r}"/>
   </xacro:thruster_macro>
   <xacro:thruster_macro namespace="${namespace}" thruster_id="2">
-   <origin xyz="0.14 -0.18515 -0.549" rpy="${0*d2r} ${0*d2r} ${0*d2r}"/>
+   <origin xyz="0 0.34 -0.21" rpy="${0*d2r} ${0*d2r} ${0*d2r}"/>
   </xacro:thruster_macro>
   <xacro:thruster_macro namespace="${namespace}" thruster_id="3">
-   <origin xyz="0.14 0.18515 -0.549" rpy="${0*d2r} ${0*d2r} ${0*d2r}"/>
+   <origin xyz="0 -0.34 -0.21" rpy="${0*d2r} ${0*d2r} ${0*d2r}"/>
   </xacro:thruster_macro>
   <xacro:thruster_macro namespace="${namespace}" thruster_id="4">
-   <origin xyz="0 0 0.549" rpy="${0*d2r} ${0*d2r} ${90.0*d2r}"/>
+   <origin xyz="0 0 0.21" rpy="${0*d2r} ${0*d2r} ${90.0*d2r}"/>
   </xacro:thruster_macro>
   <xacro:thruster_macro namespace="${namespace}" thruster_id="5">
-   <origin xyz="0 0 -0.549" rpy="${0*d2r} ${0*d2r} ${90.0*d2r}"/>
+   <origin xyz="0 0 -0.21" rpy="${0*d2r} ${0*d2r} ${90.0*d2r}"/>
   </xacro:thruster_macro>
   <xacro:thruster_macro namespace="${namespace}" thruster_id="6">
-   <origin xyz="0 -0.18515 -0.35472" rpy="${0*d2r} ${-90*d2r} ${0*d2r}"/>
+   <origin xyz="0 0.34 0" rpy="${0*d2r} ${-90*d2r} ${0*d2r}"/>
   </xacro:thruster_macro>
   <xacro:thruster_macro namespace="${namespace}" thruster_id="7">
-   <origin xyz="0 0.18515 -0.35472" rpy="${0*d2r} ${-90*d2r} ${0*d2r}"/>
+   <origin xyz="0 -0.34 0" rpy="${0*d2r} ${-90*d2r} ${0*d2r}"/>
   </xacro:thruster_macro>
 </robot>

File: Plankton/raybot_description/urdf/raybot_base.xacro (robot description, xacro)
@@ -32,9 +32,9 @@
   <!-- Parameters -->
   <xacro:property name="namespace" value="raybot"/>
-  <xacro:property name="visual_mesh_file" value="file://$(find raybot_description)/meshes/frame_kolom_origin_com.dae"/>
-  <xacro:property name="collision_mesh_file" value="file://$(find raybot_description)/meshes/frame_collision_origin_com.dae"/>
-  <xacro:property name="prop_mesh_file" value="file://$(find raybot_description)/meshes/prop.dae"/>
+  <xacro:property name="visual_mesh_file" value="file://$(find raybot_description)/meshes/raybot_simple_frame_water_v2.dae"/>
+  <xacro:property name="collision_mesh_file" value="file://$(find raybot_description)/meshes/raybot_simple_collision_v2.dae"/>
+  <xacro:property name="prop_mesh_file" value="file://$(find raybot_description)/meshes/raybot_simple_thruster_v2.dae"/>
   <!-- Mass, see p.28 in Berg2012 -->
-  <xacro:property name="mass" value="1862.87"/>
+  <xacro:property name="mass" value="40.89"/> <!-- 1862.87 of 168 xxxxxxxxxxxxxxxxxxxxxxxxxxxxxxxxxxxxxxxxxxxxxxxxxxxxxxxxxxxxxxxxxxxxxxxxxxxxxxxxxxxxxxxxxxxxxx -->
   <xacro:macro name="raybot_base" params="namespace *gazebo inertial_reference_frame">
     <!-- base_link according to ROS conventions: x forward, z up -->
@@ -43,8 +43,8 @@
         <mass value="${mass}"/>
         <origin xyz="0 0 0"/>
-        <inertia ixx="525.39" ixy="1.44" ixz="33.41" iyy="794.20" iyz="2.6" izz="691.23"/>
+        <inertia ixx="3.04999" ixy="0" ixz="0" iyy="1.19804" iyz="0" izz="2.36173"/> <!--ixx="1.19804" ixy="0" ixz="0.00124" iyy="2.36173" iyz="0" izz="3.04999" of  ixx="525.39" ixy="1.44" ixz="33.41" iyy="794.20" iyz="2.6" izz="691.23"/> of ixx="23.66" ixy="0" ixz="0" iyy="21.25" iyz="0" izz="4.6" xxxxxxxxxxxxxxxxx -->
       </inertial>
       <visual>
-        <origin xyz="0 0 0" rpy="1.5708 0 3.1416"/>
+        <origin xyz="0 0 0" rpy="0 0 0"/>
         <geometry>
           <mesh filename="${visual_mesh_file}" scale="1 1 1"/>
@@ -53,5 +53,5 @@
       <!-- bottom plate -->
       <collision>
-        <origin xyz="0 0 0" rpy="1.5708 0 3.1416"/>
+        <origin xyz="0 0 0" rpy="0 0 0"/>
         <geometry>
           <mesh filename="${collision_mesh_file}" scale="1 1 1"/>
